File: mp3/mp3_fa2026.kicad_pcb (KiCad board)
At the start: 2 copper layers, 21 x 51 mm, 41 parts, among them J1 USB4105-GF-A, J2 LEFT, J3 RIGHT, J4 DEBUG, U1 RP2354A, U2 MCP1702T-3302E_CB, X1 IQXO-791_12MHz

Commit message: finished touch ups
Routing:
- net GND: track 54.6 -> 59.1 mm, vias 37 -> 41
- net /SWCLK: track 25.4 -> 23.1 mm
- net /SWDIO: track 29.3 -> 27.9 mm
- net /GPIO16: track 24.9 -> 23.6 mm
- net /GPIO14: track 22.2 -> 21.3 mm
- net /GPIO13: track 16.6 -> 15.8 mm
- net +1V1: track 33.0 -> 32.2 mm
- net /GPIO12: track 13.3 -> 12.7 mm
- net /GPIO15: track 24.3 -> 23.8 mm
- net /GPIO11: track 10.6 -> 10.1 mm
- net /GPIO10: track 9.21 -> 8.67 mm
Other:
- board text added: "0"
- board text added: "1"
- board text added: "10"
- board text added: "11"
- board text added: "12"
- board text added: "13"
- board text added: "14"
- board text added: "15"
- board text added: "16"
- board text added: "17"
- board text added: "18"
- board text added: "19"
- board text added: "2"
- board text added: "20"
- board text added: "21"
- board text added: "22"
- board text added: "23"
- board text added: "26"
- board text added: "27"
- board text added: "28"
- board text added: "29"
- board text added: "3"
- board text added: "3V3"
- board text added: "4"
- board text added: "5"
- board text added: "6"
- board text added: "7"
- board text added: "8"
- board text added: "9"
- board text added: "BOOT"
- board text added: "GND"
- board text added: "RST"
- board text added: "Ramzey Burdette Eclectronics FA'26 Miniproject 3 - RP2354A Development Board"
- board text added: "SWCLK"
- board text added: "SWDIO"
- board text added: "VBUS"

Commit message: updated PCB
Parts:
- moved C1 2.17 mm to (181.7, 107.1), turned to -90 degrees
- moved C13 1.72 mm to (185.5, 104.5)
- moved X1 1.20 mm to (183.7, 107.5)
- moved C5 1.20 mm to (182.9, 105.5)
Routing:
- net GND: track 59.1 -> 43.4 mm, vias 41 -> 34
- net /BOOT: track 39.6 -> 46.3 mm, vias 2 -> 3
- net +3V3: track 98.8 -> 96.6 mm
- net +1V1: track 32.2 -> 30.5 mm
- net /GPIO23: track 35.9 -> 37.1 mm
- net /SWCLK: track 23.1 -> 24.1 mm
- net /SWDIO: track 27.9 -> 29.0 mm
- net Net-(U1-XIN): track 4.20 -> 5.21 mm
- net /GPIO29: track 14.5 -> 13.8 mm
Other:
- board text removed: "Ramzey Burdette Eclectronics FA'26 Miniproject 3 - RP2354A Development Board"
